File: StrainGaugeDAQ.kicad_sch (KiCad schematic)
At the start: 2 parts, among them U1 INA351CDSIDSGR, U2 MCP3562RT-E/NC

Commit message: Scem work
Parts:
- removed U1: INA351CDSIDSGR, Package_TO_SOT_SMD:TSOT-23-8, symbol AddedSymbols:INA351CDSIDSGR
Connections:
- net GND: now reaches U2.17 (DGND)
- net GND: now also U2.20 (AGND), U2.21 (GND)
- net Amp1/Vout: now reaches U2.3 (CH0)
- net Amp2/Vout: now reaches U2.4 (CH1)
- net Amp3/Vout: now reaches U2.5 (CH2)
- net Amp4/Vout: now reaches U2.6 (CH3)
Other:
- added sheet Amp1 (Amp1.kicad_sch)
- added sheet Amp2 (Amp1.kicad_sch)
- added sheet Amp3 (Amp1.kicad_sch)
- added sheet Amp4 (Amp1.kicad_sch)
- added sheet PD (PD.kicad_sch)
- moved on the sheet: U2
