File: StrainGaugeDAQ.kicad_pcb (KiCad board)
At the start: 2 copper layers, 2 parts, among them U1 INA351CDSIDSGR, U2 MCP3562RT-E/NC

Commit message: Scem work
Parts:
- added C1: C, Capacitor_SMD:C_0603_1608Metric, F.Cu at (188.0, 104.5)
- added C10: C, Capacitor_SMD:C_0603_1608Metric, F.Cu at (174.0, 90.4)
- added C11: C, Capacitor_SMD:C_0603_1608Metric, F.Cu at (174.0, 92.9)
- added C12: C, Capacitor_SMD:C_0603_1608Metric, F.Cu at (174.0, 95.4)
- added C13: C, Capacitor_SMD:C_0603_1608Metric, F.Cu at (188.0, 87.9)
- added C14: C, Capacitor_SMD:C_0603_1608Metric, F.Cu at (188.0, 90.4)
- added C15: C, Capacitor_SMD:C_0603_1608Metric, F.Cu at (188.0, 92.9)
- added C16: C, Capacitor_SMD:C_0603_1608Metric, F.Cu at (188.0, 95.4)
- added C2: C, Capacitor_SMD:C_0603_1608Metric, F.Cu at (188.0, 107.0)
- added C3: C, Capacitor_SMD:C_0603_1608Metric, F.Cu at (188.0, 109.5)
- added C4: C, Capacitor_SMD:C_0603_1608Metric, F.Cu at (188.0, 112.0)
- added C5: C, Capacitor_SMD:C_0603_1608Metric, F.Cu at (174.0, 104.5)
- added C6: C, Capacitor_SMD:C_0603_1608Metric, F.Cu at (174.0, 107.0)
- added C7: C, Capacitor_SMD:C_0603_1608Metric, F.Cu at (174.0, 109.5)
- added C8: C, Capacitor_SMD:C_0603_1608Metric, F.Cu at (174.0, 112.0)
- added C9: C, Capacitor_SMD:C_0603_1608Metric, F.Cu at (174.0, 87.9)
- added R1: R_US, Resistor_SMD:R_0603_1608Metric, F.Cu at (192.0, 104.5)
- added R10: R_US, Resistor_SMD:R_0603_1608Metric, F.Cu at (178.0, 107.0)
- added R11: R_US, Resistor_SMD:R_0603_1608Metric, F.Cu at (178.0, 109.5)
- added R12: R_US, Resistor_SMD:R_0603_1608Metric, F.Cu at (178.0, 112.0)
- added R13: R_US, Resistor_SMD:R_0603_1608Metric, F.Cu at (182.0, 104.5)
- added R14: R_US, Resistor_SMD:R_0603_1608Metric, F.Cu at (182.0, 107.0)
- added R15: R_US, Resistor_SMD:R_0603_1608Metric, F.Cu at (182.0, 109.5)
- added R16: R_US, Resistor_SMD:R_0603_1608Metric, F.Cu at (182.0, 112.0)
- added R17: R_US, Resistor_SMD:R_0603_1608Metric, F.Cu at (178.0, 87.9)
- added R18: R_US, Resistor_SMD:R_0603_1608Metric, F.Cu at (178.0, 90.4)
- added R19: R_US, Resistor_SMD:R_0603_1608Metric, F.Cu at (178.0, 92.9)
- added R2: R_US, Resistor_SMD:R_0603_1608Metric, F.Cu at (192.0, 107.0)
- added R20: R_US, Resistor_SMD:R_0603_1608Metric, F.Cu at (178.0, 95.4)
- added R21: R_US, Resistor_SMD:R_0603_1608Metric, F.Cu at (182.0, 87.9)
- added R22: R_US, Resistor_SMD:R_0603_1608Metric, F.Cu at (182.0, 90.4)
- added R23: R_US, Resistor_SMD:R_0603_1608Metric, F.Cu at (182.0, 92.9)
- added R24: R_US, Resistor_SMD:R_0603_1608Metric, F.Cu at (182.0, 95.4)
- added R25: R_US, Resistor_SMD:R_0603_1608Metric, F.Cu at (192.0, 87.9)
- added R26: R_US, Resistor_SMD:R_0603_1608Metric, F.Cu at (192.0, 90.4)
- added R27: R_US, Resistor_SMD:R_0603_1608Metric, F.Cu at (192.0, 92.9)
- added R28: R_US, Resistor_SMD:R_0603_1608Metric, F.Cu at (192.0, 95.4)
- added R29: R_US, Resistor_SMD:R_0603_1608Metric, F.Cu at (196.0, 87.9)
- added R3: R_US, Resistor_SMD:R_0603_1608Metric, F.Cu at (192.0, 109.5)
- added R30: R_US, Resistor_SMD:R_0603_1608Metric, F.Cu at (196.0, 90.4)
- added R31: R_US, Resistor_SMD:R_0603_1608Metric, F.Cu at (196.0, 92.9)
- added R32: R_US, Resistor_SMD:R_0603_1608Metric, F.Cu at (196.0, 95.4)
- added R4: R_US, Resistor_SMD:R_0603_1608Metric, F.Cu at (192.0, 112.0)
- added R5: R_US, Resistor_SMD:R_0603_1608Metric, F.Cu at (196.0, 104.5)
- added R6: R_US, Resistor_SMD:R_0603_1608Metric, F.Cu at (196.0, 107.0)
- added R7: R_US, Resistor_SMD:R_0603_1608Metric, F.Cu at (196.0, 109.5)
- added R8: R_US, Resistor_SMD:R_0603_1608Metric, F.Cu at (196.0, 112.0)
- added R9: R_US, Resistor_SMD:R_0603_1608Metric, F.Cu at (178.0, 104.5)
- added U3: INA351CDSIDSGR, Package_TO_SOT_SMD:TSOT-23-8, F.Cu at (174.5, 115.7)
- added U4: INA351CDSIDSGR, Package_TO_SOT_SMD:TSOT-23-8, F.Cu at (174.5, 99.0)
- added U5: INA351CDSIDSGR, Package_TO_SOT_SMD:TSOT-23-8, F.Cu at (188.6, 99.0)
- moved U1 41.8 mm to (188.6, 115.7)
Connections:
- U1 pad 1: unconnected-(U1-GS-Pad1) -> Net-(U1-GS)
- U1 pad 2: unconnected-(U1-IN--Pad2) -> /Amp1/In+
- U1 pad 3: unconnected-(U1-IN+-Pad3) -> Net-(U1-IN+)
- U1 pad 4: unconnected-(U1-V--Pad4) -> GND
- U1 pad 5: unconnected-(U1-REF-Pad5) -> Net-(U1-REF)
- U1 pad 6: unconnected-(U1-OUT-Pad6) -> Net-(U1-OUT)
- U1 pad 7: unconnected-(U1-V+-Pad7) -> /Amp1/AVin
- U1 pad 8: unconnected-(U1-*SHDN-Pad8) -> /Amp1/AVin
- U2 pad 17: unconnected-(U2-DGND-Pad17) -> GND
- U2 pad 20: unconnected-(U2-AGND-Pad20) -> GND
- U2 pad 21: unconnected-(U2-GND-Pad21) -> GND
- U2 pad 3: unconnected-(U2-CH0-Pad3) -> /Amp1/Vout
- U2 pad 4: unconnected-(U2-CH1-Pad4) -> /Amp2/Vout
- U2 pad 5: unconnected-(U2-CH2-Pad5) -> /Amp3/Vout
- U2 pad 6: unconnected-(U2-CH3-Pad6) -> /Amp4/Vout

Commit message: Schematic done
Parts:
- added C17: C, Capacitor_SMD:C_0603_1608Metric, F.Cu at (168.5, 81.0)
- added C18: C, Capacitor_SMD:C_0603_1608Metric, F.Cu at (201.1, 79.0)
- added C19: C, Capacitor_SMD:C_0603_1608Metric, F.Cu at (189.1, 79.0)
- added C20: C, Capacitor_SMD:C_0603_1608Metric, F.Cu at (195.1, 79.0)
- added C21: C, Capacitor_SMD:C_0603_1608Metric, F.Cu at (189.1, 59.0)
- added C22: C, Capacitor_SMD:C_0603_1608Metric, F.Cu at (189.1, 61.5)
- added C23: C, Capacitor_SMD:C_0603_1608Metric, F.Cu at (189.1, 64.0)
- added C24: 100n, Capacitor_SMD:C_0603_1608Metric, F.Cu at (189.1, 66.6)
- added C25: 22u, Capacitor_SMD:C_0603_1608Metric, F.Cu at (189.1, 69.1)
- added C27: 100n, Capacitor_SMD:C_0603_1608Metric, F.Cu at (189.1, 71.6)
- added C28: 100n, Capacitor_SMD:C_0603_1608Metric, F.Cu at (193.1, 59.0)
- added C29: 10u, Capacitor_SMD:C_0603_1608Metric, F.Cu at (193.1, 61.5)
- added C30: 10u, Capacitor_SMD:C_0603_1608Metric, F.Cu at (193.1, 64.0)
- added C31: 100n, Capacitor_SMD:C_0603_1608Metric, F.Cu at (193.1, 66.6)
- added C32: 100n, Capacitor_SMD:C_0603_1608Metric, F.Cu at (193.1, 69.1)
- added C33: 100n, Capacitor_SMD:C_0603_1608Metric, F.Cu at (193.1, 71.6)
- added C34: 100n, Capacitor_SMD:C_0603_1608Metric, F.Cu at (197.1, 59.0)
- added C35: 100n, Capacitor_SMD:C_0603_1608Metric, F.Cu at (197.1, 61.5)
- added C37: 100n, Capacitor_SMD:C_0603_1608Metric, F.Cu at (174.5, 59.0)
- added C38: 10u, Capacitor_SMD:C_0603_1608Metric, F.Cu at (174.5, 61.5)
- added C39: 100n, Capacitor_SMD:C_0603_1608Metric, F.Cu at (174.5, 64.0)
- added C40: 10u, Capacitor_SMD:C_0603_1608Metric, F.Cu at (174.5, 66.6)
- added FB1: FerriteBead, Inductor_SMD:L_0603_1608Metric, F.Cu at (197.1, 64.0)
- added FB2: FerriteBead, Inductor_SMD:L_0603_1608Metric, F.Cu at (174.5, 69.1)
- added J1: IN1, AA-Custom:SolderPad_01x02, F.Cu at (169.5, 59.8)
- added J2: IN2, AA-Custom:SolderPad_01x02, F.Cu at (169.5, 63.8)
- added J3: IN3, AA-Custom:SolderPad_01x02, F.Cu at (169.5, 67.8)
- added J4: IN4, AA-Custom:SolderPad_01x02, F.Cu at (169.5, 71.8)
- added J5: VBAT, AA-Custom:SolderPad_01x02, F.Cu at (169.5, 75.8)
- added J6: SPI+INT, Connector_PinHeader_2.54mm:PinHeader_1x05_P2.54mm_Vertical, F.Cu at (182.8, 60.1)
- added L1: 3.3u, Inductor_SMD:L_Vishay_IFSC-1515AH_4x4x1.8mm, F.Cu at (201.9, 69.8)
- added R33: 52.3k, Resistor_SMD:R_0603_1608Metric, F.Cu at (197.1, 66.6)
- added R34: 10k, Resistor_SMD:R_0603_1608Metric, F.Cu at (197.1, 69.1)
- added R36: 10, Resistor_SMD:R_0603_1608Metric, F.Cu at (174.5, 71.6)
- added R37: 10, Resistor_SMD:R_0603_1608Metric, F.Cu at (178.5, 59.0)
- added R38: 10, Resistor_SMD:R_0603_1608Metric, F.Cu at (178.5, 61.5)
- added R39: 10, Resistor_SMD:R_0603_1608Metric, F.Cu at (178.5, 64.0)
- added R40: 10k, Resistor_SMD:R_0603_1608Metric, F.Cu at (178.5, 66.6)
- added R41: 10, Resistor_SMD:R_0603_1608Metric, F.Cu at (178.5, 69.1)
- added U6: AP62150Z6, Package_TO_SOT_SMD:SOT-563, F.Cu at (200.8, 74.3)
- added U7: AP2127K-3.3, Package_TO_SOT_SMD:SOT-23-5, F.Cu at (201.7, 60.2)
- added U8: AP2127K-3.3, Package_TO_SOT_SMD:SOT-23-5, F.Cu at (201.7, 64.8)
Connections:
- C10 pad 1: /Amp3/AVin -> AVDD
- C13 pad 1: /Amp4/AVin -> AVDD
- C14 pad 1: /Amp4/AVin -> AVDD
- C2 pad 1: /Amp1/AVin -> AVDD
- C3 pad 1: /Amp1/AVin -> AVDD
- C5 pad 1: /Amp2/AVin -> AVDD
- C6 pad 1: /Amp2/AVin -> AVDD
- C9 pad 1: /Amp3/AVin -> AVDD
- R1 pad 1: /Amp1/AVin -> AVDD
- R11 pad 1: /Amp2/AVin -> AVDD
- R14 pad 1: /Amp2/AVin -> AVDD
- R17 pad 1: /Amp3/AVin -> AVDD
- R19 pad 1: /Amp3/AVin -> AVDD
- R2 pad 1: /Amp1/AVin -> AVDD
- R22 pad 1: /Amp3/AVin -> AVDD
- R25 pad 1: /Amp4/AVin -> AVDD
- R27 pad 1: /Amp4/AVin -> AVDD
- R30 pad 1: /Amp4/AVin -> AVDD
- R4 pad 1: /Amp1/AVin -> AVDD
- R9 pad 1: /Amp2/AVin -> AVDD
- U1 pad 7: /Amp1/AVin -> AVDD
- U1 pad 8: /Amp1/AVin -> AVDD
- U2 pad 1: unconnected-(U2-REFIN--Pad1) -> Net-(U2-AGND)
- U2 pad 11: unconnected-(U2-*CS-Pad11) -> Net-(U2-*CS)
- U2 pad 12: unconnected-(U2-SCK-Pad12) -> Net-(U2-SCK)
- U2 pad 13: unconnected-(U2-SDI-Pad13) -> Net-(U2-SDI)
- U2 pad 14: unconnected-(U2-SDO-Pad14) -> Net-(U2-SDO)
- U2 pad 15: unconnected-(U2-*IRQ/MDAT-Pad15) -> Net-(U2-*IRQ/MDAT)
- U2 pad 18: unconnected-(U2-DVDD-Pad18) -> DVDD
- U2 pad 19: unconnected-(U2-AVDD-Pad19) -> AVDD
- U2 pad 2: unconnected-(U2-REFIN+/OUT-Pad2) -> AVDD
- U2 pad 20: GND -> Net-(U2-AGND)
- U3 pad 7: /Amp2/AVin -> AVDD
- U3 pad 8: /Amp2/AVin -> AVDD
- U4 pad 7: /Amp3/AVin -> AVDD
- U4 pad 8: /Amp3/AVin -> AVDD
- U5 pad 7: /Amp4/AVin -> AVDD
- U5 pad 8: /Amp4/AVin -> AVDD
Other:
- board outline added: 86.6 x 69.5 mm

Commit message: Layout work
Parts:
- removed FB2: FerriteBead, Inductor_SMD:L_0603_1608Metric
- removed R12, R13, R20, R21, R28, R29, R6, R7: R_US, Resistor_SMD:R_0603_1608Metric
- C1, C10, C11, C13, C14, C15, C17, C18, C19, C2, C20, C3, C5, C6, C7, C9: value C -> 100n; moved to B.Cu
- C21, C22: value C -> 22u
- C23: value C -> 100n
- C25, C27, C30, C31, C32, C34, C37, C38, C39, C40, R17, R2, R25, R33, R34, R9: moved to B.Cu
- J5: value VBAT -> 6-18V
- R14, R15, R22, R23, R30, R31, R4, R5: value R_US -> 10k; moved to B.Cu
- moved C20 59.1 mm to (146.5, 112.6), turned to 90 degrees
- moved R3 57.4 mm to (141.4, 82.3), turned to 180 degrees
- moved R25 56.5 mm to (141.9, 114.1), turned to -90 degrees
- moved R26 56.5 mm to (141.1, 114.9), turned to 180 degrees
- moved R1 56.2 mm to (141.4, 80.0), turned to 180 degrees
- moved R8 56.2 mm to (149.2, 81.0), turned to 180 degrees
- moved R2 55.9 mm to (142.3, 81.4), turned to -90 degrees
- moved C18 55.3 mm to (146.9, 90.1), turned to 90 degrees
- moved U1 55.1 mm to (145.6, 81.2)
- moved R27 54.6 mm to (141.1, 112.5), turned to 180 degrees
- moved R4 53.8 mm to (149.2, 79.5)
- moved J4 53.7 mm to (136.3, 114.0), turned to 90 degrees
- moved J6 52.5 mm to (170.9, 111.2), turned to 180 degrees
- moved R5 52.4 mm to (149.2, 81.0), turned to 180 degrees
- moved U7 52.3 mm to (159.6, 91.2), turned to -90 degrees
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Connections:
- U1 pad 1: Net-(U1-GS) -> unconnected-(U1-GS-Pad1)
- U2 pad 1: Net-(U2-AGND) -> GND
- U2 pad 20: Net-(U2-AGND) -> GND
- U3 pad 1: Net-(U3-GS) -> unconnected-(U3-GS-Pad1)
- U4 pad 1: Net-(U4-GS) -> unconnected-(U4-GS-Pad1)
- U5 pad 1: Net-(U5-GS) -> unconnected-(U5-GS-Pad1)
Routing:
- net GND: track 0.00 -> 40.2 mm, vias 0 -> 50
- net 5V: track 0.00 -> 23.4 mm, vias 0 -> 5
- net DVDD: track 0.00 -> 8.57 mm, vias 0 -> 2
- net /Amp1/In+: track 0.00 -> 8.51 mm
- net /Amp2/In+: track 0.00 -> 8.45 mm
- net /Amp3/In+: track 0.00 -> 8.06 mm
- net /Amp4/In+: track 0.00 -> 7.83 mm
- net Net-(U1-REF): track 0.00 -> 7.46 mm, vias 0 -> 1
- net Net-(U5-REF): track 0.00 -> 7.26 mm, vias 0 -> 1
- net Net-(U4-REF): track 0.00 -> 7.10 mm, vias 0 -> 1
- net Net-(U3-REF): track 0.00 -> 6.99 mm, vias 0 -> 1
- net Net-(U1-IN+): track 0.00 -> 4.48 mm, vias 0 -> 1
- net Net-(U3-IN+): track 0.00 -> 3.62 mm, vias 0 -> 1
- net AVDD: track 0.00 -> 3.55 mm, vias 0 -> 4
- net Net-(U4-IN+): track 0.00 -> 3.28 mm, vias 0 -> 1
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- added copper zone on F.Cu, net /PD/VCC
- added copper zone on B.Cu, net 5V
- added copper zone on F.Cu, net 5V
- added copper zone on B.Cu, net AVDD
- added copper zone on F.Cu, net AVDD
- added copper zone on B.Cu, net GND
- added copper zone on F.Cu, net GND
- added copper zone on F.Cu, net Net-(U6-EN)
- added copper zone on F.Cu, net Net-(U6-SW)
Other:
- board size 86.6 x 69.5 mm -> 39.3 x 62.7 mm
- board text added: "CS"
- board text added: "GND"
- board text added: "IRQ"
- board text added: "SCLK"
- board text added: "SDI"
- board text added: "SDO"

Commit message: fab files created
Parts:
- added H1: MountingScrew, AA-Custom:EyePicture, F.Cu at (153.1, 73.2)
- added H2: MountingScrew, AA-Custom:EyePicture, F.Cu at (153.1, 112.3)
- moved C15 8.15 mm to (146.5, 106.7)
- moved C16 8.15 mm to (148.7, 106.7)
- moved J4 8.15 mm to (136.3, 105.9)
- moved U5 8.15 mm to (144.9, 105.7)
- moved C13 8.15 mm to (143.4, 104.4)
- moved C14 8.15 mm to (144.9, 104.4)
- moved C20 8.15 mm to (146.5, 104.4)
- moved R25 8.15 mm to (141.9, 105.9)
- moved R26 8.15 mm to (141.1, 106.8)
- moved R27 8.15 mm to (141.1, 104.4)
- moved R30 8.15 mm to (148.8, 103.6)
- moved R31 8.15 mm to (148.7, 105.1)
- moved R32 8.15 mm to (148.7, 105.1)
- moved C10 6.15 mm to (145.0, 96.0)
- moved C11 6.15 mm to (146.8, 98.3)
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Routing:
- net AVDD: track 3.55 -> 72.5 mm, vias 4 -> 20
- net /Amp1/Vout: track 1.54 -> 28.6 mm
- net /Amp2/Vout: track 1.55 -> 21.0 mm
- net /Amp3/Vout: track 0.00 -> 13.8 mm
- net /Amp4/Vout: track 1.55 -> 12.7 mm
- net DVDD: track 8.57 -> 19.7 mm
- net Net-(U2-*IRQ/MDAT): track 0.00 -> 6.51 mm
- net Net-(U2-*CS): track 0.00 -> 5.02 mm
- net Net-(U2-SCK): track 0.00 -> 4.97 mm
- net Net-(U2-SDO): track 0.00 -> 4.97 mm
- net Net-(U2-SDI): track 0.00 -> 4.97 mm
- net Net-(J6-Pin_5): track 0.00 -> 4.55 mm
- net Net-(J6-Pin_4): track 0.00 -> 3.56 mm
- net Net-(J6-Pin_1): track 0.00 -> 3.56 mm
- net Net-(J6-Pin_2): track 0.00 -> 3.54 mm
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Other:
- board size 39.3 x 62.7 mm -> 39.4 x 50.7 mm
- board text added: "Double Barrel Eye Strain Design by Nick Lee 6/7/26"
