File: Amp1.kicad_sch (KiCad schematic)
At the start: 14 parts, among them U1 INA351CDSIDSGR

Commit message: Layout work
Parts:
- removed R6, R7: R_US, Resistor_SMD:R_0603_1608Metric, symbol Device:R_US
- C1, C17, C2, C3: value C -> 100n
- R4, R5: value R_US -> 10k
Connections:
- no-connect marks 0 -> 1

Commit message: BOM generated
Parts:
- C1, C17, C2, C3: digikey (none) -> 1276-1000-1-ND
- C4: value C -> 100n; digikey (none) -> 1276-1000-1-ND
- R1, R2: value R_US -> 350; digikey (none) -> 738-RNCF0603DTE348RCT-ND
- R3, R8: value R_US -> 120; digikey (none) -> 541-10426-1-ND
- R4, R5: digikey (none) -> 311-10.0KHRCT-ND
Changed lines of the file:
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@@
 			)
 		)
-		(property "Value" "R_US"
+		(property "Value" "350"
 			(at 120.65 92.7099 0)
 			(show_name no)
@@
 		)
 		(property "Description" "Resistor, US symbol"
+			(at 118.11 91.44 0)
+			(hide yes)
+			(show_name no)
+			(do_not_autoplace no)
+			(effects
+				(font
+					(size 1.27 1.27)
+				)
+			)
+		)
+		(property "digikey" "738-RNCF0603DTE348RCT-ND"
 			(at 118.11 91.44 0)
 			(hide yes)
@@
 			)
 		)
+		(property "digikey" "311-10.0KHRCT-ND"
+			(at 160.02 64.77 90)
+			(hide yes)
+			(show_name no)
+			(do_not_autoplace no)
+			(effects
+				(font
+					(size 1.27 1.27)
+				)
+			)
+		)
 		(pin "2"
 		)
@@
 		(property "Description" "Unpolarized capacitor"
 			(at 171.45 73.66 0)
+			(hide yes)
+			(show_name no)
+			(do_not_autoplace no)
+			(effects
+				(font
+					(size 1.27 1.27)
+				)
+			)
+		)
+		(property "digikey" "1276-1000-1-ND"
+			(at 171.45 73.66 90)
 			(hide yes)
 			(show_name no)
@@
 			)
 		)
+		(property "digikey" "311-10.0KHRCT-ND"
+			(at 170.18 64.77 90)
+			(hide yes)
+			(show_name no)
+			(do_not_autoplace no)
+			(effects
+				(font
+					(size 1.27 1.27)
+				)
+			)
+		)
 		(pin "2"
 		)
@@
 			)
 		)
-		(property "Value" "C"
+		(property "Value" "100n"
 			(at 195.58 104.1399 0)
 			(show_name no)
@@
 		)
 		(property "Description" "Unpolarized capacitor"
+			(at 191.77 102.87 0)
+			(hide yes)
+			(show_name no)
+			(do_not_autoplace no)
+			(effects
+				(font
+					(size 1.27 1.27)
+				)
+			)
+		)
+		(property "digikey" "1276-1000-1-ND"
 			(at 191.77 102.87 0)
 			(hide yes)
@@
 			)
 		)
+		(property "digikey" "1276-1000-1-ND"
+			(at 99.06 81.28 0)
+			(hide yes)
+			(show_name no)
+			(do_not_autoplace no)
+			(effects
+				(font
+					(size 1.27 1.27)
+				)
+			)
+		)
 		(pin "2"
 		)
@@
 			)
 		)
-		(property "Value" "R_US"
+		(property "Value" "120"
 			(at 182.88 92.71 90)
 			(show_name no)
@@
 		(property "Description" "Resistor, US symbol"
 			(at 182.88 96.52 0)
+			(hide yes)
+			(show_name no)
+			(do_not_autoplace no)
+			(effects
+				(font
+					(size 1.27 1.27)
+				)
+			)
+		)
+		(property "digikey" "541-10426-1-ND"
+			(at 182.88 96.52 90)
 			(hide yes)
 			(show_name no)
@@
 		(property "Description" "Unpolarized capacitor"
 			(at 146.05 73.66 0)
+			(hide yes)
+			(show_name no)
+			(do_not_autoplace no)
+			(effects
+				(font
+					(size 1.27 1.27)
+				)
+			)
+		)
+		(property "digikey" "1276-1000-1-ND"
+			(at 146.05 73.66 90)
 			(hide yes)
 			(show_name no)
@@
 			)
 		)
-		(property "Value" "R_US"
+		(property "Value" "120"
 			(at 110.49 105.4099 0)
 			(show_name no)
@@
 		)
 		(property "Description" "Resistor, US symbol"
+			(at 107.95 104.14 0)
+			(hide yes)
+			(show_name no)
+			(do_not_autoplace no)
+			(effects
+				(font
+					(size 1.27 1.27)
+				)
+			)
+		)
+		(property "digikey" "541-10426-1-ND"
 			(at 107.95 104.14 0)
 			(hide yes)
@@
 			)
 		)
+		(property "digikey" "1276-1000-1-ND"
+			(at 88.9 81.28 0)
+			(hide yes)
+			(show_name no)
+			(do_not_autoplace no)
+			(effects
+				(font
+					(size 1.27 1.27)
+				)
+			)
+		)
 		(pin "2"
 		)
@@
 			)
 		)
-		(property "Value" "R_US"
+		(property "Value" "350"
 			(at 110.49 92.7099 0)
 			(show_name no)
@@
 			(at 107.95 91.44 0)
 			(hide yes)
+			(show_name no)
+			(do_not_autoplace no)
+			(effects
+				(font
+					(size 1.27 1.27)
+				)
+			)
+		)
+		(property "digikey" "738-RNCF0603DTE348RCT-ND"
+			(at 107.95 91.44 0)
+			(hide yes)
